File: hardware/vango-pcb/vango-pcb.kicad_sch (KiCad schematic)
At the start: 13 parts, among them J1 XT60PW-M, J2 NeoPixel, J3 I2C, J4 Conn_01x07, J5 SPI, J6 Conn_01x02, SW1 SW_SPDT, U1 MD41B, U2 REG15D, U3 MD41B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

Commit message: add servo connector, more space for voltage reg
Parts:
- removed J4: Conn_01x07, Connector_PinHeader_2.54mm:PinHeader_1x07_P2.54mm_Vertical, symbol Connector_Generic:Conn_01x07
- added J7: Conn_01x02, Connector_PinHeader_2.54mm:PinHeader_1x02_P2.54mm_Vertical, symbol Connector_Generic:Conn_01x02
- added J8: SG90_Servo, Connector_PinHeader_2.54mm:PinHeader_1x03_P2.54mm_Vertical, symbol Connector_Generic:Conn_01x03
Connections:
- net GNDPWR is gone; now on net GND: J2.3 (Pin_3), U1.9 (GND), U2.4 (GND), U3.9 (GND)
- net +5V: now also J7.2 (Pin_2), J8.2 (Pin_2)
- net A8: now also J8.3 (Pin_3)
- net GND: now also J7.1 (Pin_1), J8.1 (Pin_1)

Commit message: pcb should be all good now
Parts:
- added J4: Conn_01x06, Connector_PinHeader_2.54mm:PinHeader_1x06_P2.54mm_Vertical, symbol Connector_Generic:Conn_01x06
- added J9: Conn_01x02, Connector_PinHeader_2.54mm:PinHeader_1x02_P2.54mm_Vertical, symbol Connector_Generic:Conn_01x02
Connections:
- net +3V3: now also J9.1 (Pin_1)
- net A0: now also J4.1 (Pin_1)
- net A1: now also J4.2 (Pin_2)
- net A2: now also J4.3 (Pin_3)
- net A3: now also J4.4 (Pin_4)
- net A4: now also J4.5 (Pin_5)
- net A5: now also J4.6 (Pin_6)
- net GND: now also J1.1 (-), U2.3 (GND), J9.2 (Pin_2)
- net at SW1.3 (C): now also J1.2 (+); no longer J1.1 (+)
Other:
- moved on the sheet: J1, J6, J7, SW1, U2
